File: Swadge-S2-Devkit/Swadge-S2-Devkit.kicad_sch (KiCad schematic)
At the start: 90 parts, among them J7 LEDK_J, J8 LCD18, J9 LCD28, P1 USB_C_Plug_USB2.0, Q4 AP2003_PN_FET, SW1 TS-1109S-A-A, SW2 TS-1109S-A-A, SW3 TS-1109S-A-A, SW4 TS-1109S-A-A, SW5 TS-1109S-A-A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

Commit message: Fixed footprints and models for mic, bzr, slide switch, SK6812
Parts:
- D1, D10, D2, D3, D4, D5, D6, D7: footprint Swadge_Parts:SK6812SIDE -> Swadge_Parts:SK6812_SIDE_2
- LS1: footprint Swadge_Parts:Buzzer_12x9.5RM7.6 -> Swadge_Parts:Buzzer_12.5x7.5
- MK1: footprint Swadge_Parts:CMA-4544PF-W -> Swadge_Parts:INGHAi GMI6050P-56DB
Changed lines of the file:
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@@
       (effects (font (size 1.27 1.27)) (justify left))
     )
-    (property "Footprint" "Swadge_Parts:Buzzer_12x9.5RM7.6" (id 2) (at 237.49 80.01 0)
+    (property "Footprint" "Swadge_Parts:Buzzer_12.5x7.5" (id 2) (at 237.49 80.01 0)
       (effects (font (size 1.27 1.27)) hide)
     )
@@
     (pin "1")
   )
-  (symbol (lib_name "SK6812SIDE_3") (lib_id "Swadge_Parts:SK6812SIDE") (at 58.42 138.43 0) (unit 1)
+  (symbol (lib_id "Swadge_Parts:SK6812SIDE") (at 58.42 138.43 0) (unit 1)
     (in_bom yes) (on_board yes)
     (property "Reference" "D3" (id 0) (at 62.23 130.81 0)
@@
       (effects (font (size 1.524 1.524)))
     )
-    (property "Footprint" "Swadge_Parts:SK6812SIDE" (id 2) (at 58.42 128.27 0)
+    (property "Footprint" "Swadge_Parts:SK6812_SIDE_2" (id 2) (at 58.42 128.27 0)
       (effects (font (size 1.524 1.524)) hide)
     )
@@
       (effects (font (size 1.524 1.524)))
     )
-    (property "Footprint" "Swadge_Parts:SK6812SIDE" (id 2) (at 140.97 128.27 0)
+    (property "Footprint" "Swadge_Parts:SK6812_SIDE_2" (id 2) (at 140.97 128.27 0)
       (effects (font (size 1.524 1.524)) hide)
     )
@@
     )
     (property "Value" "Microphone" (id 1) (at 256.54 44.45 0))
-    (property "Footprint" "Swadge_Parts:CMA-4544PF-W" (id 2) (at 248.92 44.45 90)
+    (property "Footprint" "Swadge_Parts:INGHAi GMI6050P-56DB" (id 2) (at 248.92 44.45 90)
       (effects (font (size 1.27 1.27)) hide)
     )
@@
       (effects (font (size 1.524 1.524)))
     )
-    (property "Footprint" "Swadge_Parts:SK6812SIDE" (id 2) (at 124.46 128.27 0)
+    (property "Footprint" "Swadge_Parts:SK6812_SIDE_2" (id 2) (at 124.46 128.27 0)
       (effects (font (size 1.524 1.524)) hide)
     )
@@
       (effects (font (size 1.524 1.524)))
     )
-    (property "Footprint" "Swadge_Parts:SK6812SIDE" (id 2) (at 91.44 128.27 0)
+    (property "Footprint" "Swadge_Parts:SK6812_SIDE_2" (id 2) (at 91.44 128.27 0)
       (effects (font (size 1.524 1.524)) hide)
     )
@@
       (effects (font (size 1.524 1.524)))
     )
-    (property "Footprint" "Swadge_Parts:SK6812SIDE" (id 2) (at 107.95 128.27 0)
+    (property "Footprint" "Swadge_Parts:SK6812_SIDE_2" (id 2) (at 107.95 128.27 0)
       (effects (font (size 1.524 1.524)) hide)
     )
@@
       (effects (font (size 1.524 1.524)))
     )
-    (property "Footprint" "Swadge_Parts:SK6812SIDE" (id 2) (at 25.4 128.27 0)
+    (property "Footprint" "Swadge_Parts:SK6812_SIDE_2" (id 2) (at 25.4 128.27 0)
       (effects (font (size 1.524 1.524)) hide)
     )
@@
       (effects (font (size 1.524 1.524)))
     )
-    (property "Footprint" "Swadge_Parts:SK6812SIDE" (id 2) (at 74.93 128.27 0)
+    (property "Footprint" "Swadge_Parts:SK6812_SIDE_2" (id 2) (at 74.93 128.27 0)
       (effects (font (size 1.524 1.524)) hide)
     )
@@
       (effects (font (size 1.524 1.524)))
     )
-    (property "Footprint" "Swadge_Parts:SK6812SIDE" (id 2) (at 41.91 128.27 0)
+    (property "Footprint" "Swadge_Parts:SK6812_SIDE_2" (id 2) (at 41.91 128.27 0)
       (effects (font (size 1.524 1.524)) hide)
     )
@@
       (effects (font (size 1.27 1.27)) hide)
     )
-    (property "LCSC" "C22452" (id 7) (at 67.31 170.18 0)
+    (property "LCSC" "C22452" (id 8) (at 67.31 170.18 0)
       (effects (font (size 1.27 1.27)) hide)
     )
@@
     )
     (path "/600449c1-75c9-4c5e-bdff-37bb5ef723e1"
-      (reference "D1") (unit 1) (value "SK6812SIDE") (footprint "Swadge_Parts:SK6812SIDE")
+      (reference "D1") (unit 1) (value "SK6812SIDE") (footprint "Swadge_Parts:SK6812_SIDE_2")
     )
     (path "/b425d9db-05e1-4ce5-8e86-6b4fad1f09b2"
-      (reference "D2") (unit 1) (value "SK6812SIDE") (footprint "Swadge_Parts:SK6812SIDE")
+      (reference "D2") (unit 1) (value "SK6812SIDE") (footprint "Swadge_Parts:SK6812_SIDE_2")
     )
     (path "/18d3b882-ee49-4dd2-b2fb-6cac35ccc9cc"
-      (reference "D3") (unit 1) (value "SK6812SIDE") (footprint "Swadge_Parts:SK6812SIDE")
+      (reference "D3") (unit 1) (value "SK6812SIDE") (footprint "Swadge_Parts:SK6812_SIDE_2")
     )
     (path "/90b780aa-ec00-4512-8bd4-ea6d7a4b0bfe"
-      (reference "D4") (unit 1) (value "SK6812SIDE") (footprint "Swadge_Parts:SK6812SIDE")
+      (reference "D4") (unit 1) (value "SK6812SIDE") (footprint "Swadge_Parts:SK6812_SIDE_2")
     )
     (path "/3ac74900-a722-4894-aa95-bda370a2a7ce"
-      (reference "D5") (unit 1) (value "SK6812SIDE") (footprint "Swadge_Parts:SK6812SIDE")
+      (reference "D5") (unit 1) (value "SK6812SIDE") (footprint "Swadge_Parts:SK6812_SIDE_2")
     )
     (path "/55810db0-3a0f-41a9-893b-cb106d640f20"
-      (reference "D6") (unit 1) (value "SK6812SIDE") (footprint "Swadge_Parts:SK6812SIDE")
+      (reference "D6") (unit 1) (value "SK6812SIDE") (footprint "Swadge_Parts:SK6812_SIDE_2")
     )
     (path "/306a2ccc-4f78-4c7c-88ed-3980a2a5fa2b"
-      (reference "D7") (unit 1) (value "SK6812SIDE") (footprint "Swadge_Parts:SK6812SIDE")
+      (reference "D7") (unit 1) (value "SK6812SIDE") (footprint "Swadge_Parts:SK6812_SIDE_2")
     )
     (path "/3bf538f9-0e4b-4f29-800e-3918debddaf4"
@@
     )
     (path "/269738b8-ce1c-4500-8039-88ec03ba0178"
-      (reference "D10") (unit 1) (value "SK6812SIDE") (footprint "Swadge_Parts:SK6812SIDE")
+      (reference "D10") (unit 1) (value "SK6812SIDE") (footprint "Swadge_Parts:SK6812_SIDE_2")
     )
     (path "/473ba183-06de-4417-adf9-410137ae10e9"
@@
     )
     (path "/14c9349a-f0fb-4244-9f6f-4c73e3e70cf2"
-      (reference "LS1") (unit 1) (value "Buzzer") (footprint "Swadge_Parts:Buzzer_12x9.5RM7.6")
+      (reference "LS1") (unit 1) (value "Buzzer") (footprint "Swadge_Parts:Buzzer_12.5x7.5")
     )
     (path "/29767c92-4da0-4b29-b6b0-eff8635f995d"
-      (reference "MK1") (unit 1) (value "Microphone") (footprint "Swadge_Parts:CMA-4544PF-W")
+      (reference "MK1") (unit 1) (value "Microphone") (footprint "Swadge_Parts:INGHAi GMI6050P-56DB")
     )
     (path "/51601e67-514c-4451-9a6d-296311e33e63"

Commit message: Added correct FPC connector footprint
Parts:
- U14: footprint Swadge_Parts:FH26W-15S-0.3SHW(60) -> Swadge_Parts:HCTL HC-FPC-03-10-15RLTAG
Changed lines of the file:
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@@
     (property "Reference" "U14" (id 0) (at 311.15 64.77 0))
     (property "Value" "RB017A1505A_Connector" (id 1) (at 311.15 67.31 0))
-    (property "Footprint" "Swadge_Parts:FH26W-15S-0.3SHW(60)" (id 2) (at 311.15 53.34 0)
+    (property "Footprint" "Swadge_Parts:HCTL HC-FPC-03-10-15RLTAG" (id 2) (at 311.15 53.34 0)
       (effects (font (size 1.27 1.27)) hide)
     )
@@
     )
     (path "/96104548-f9fc-4434-8156-41330e2ddd6c"
-      (reference "U14") (unit 1) (value "RB017A1505A_Connector") (footprint "Swadge_Parts:FH26W-15S-0.3SHW(60)")
+      (reference "U14") (unit 1) (value "RB017A1505A_Connector") (footprint "Swadge_Parts:HCTL HC-FPC-03-10-15RLTAG")
     )
     (path "/bb2dd9fb-8760-4d91-aa67-00ca9845376c"

Commit message: Update main board
Parts:
- removed J7: LEDK_J, Swadge_Parts:PinHeader_1x02_P2.54mm_Vertical, symbol Swadge_Parts:Conn_01x02_Male
- removed J8: LCD18, Swadge_Parts:PinHeader_1x03_P2.54mm_Vertical, symbol Swadge_Parts:Conn_01x03_Male
- removed J9: LCD28, Swadge_Parts:PinHeader_1x03_P2.54mm_Vertical, symbol Swadge_Parts:Conn_01x03_Male
- removed L2: 100uH, Swadge_Parts:L_1210_3225Metric, symbol Swadge_Parts:L
- removed Q4: AP2003_PN_FET, Swadge_Parts:SOT-23-6, symbol Swadge_Parts:AP2003_PN_FET
- removed R10: 10Ω, Swadge_Parts:R_0603_1608Metric, symbol Swadge_Parts:R_US
- removed U4: GS321-TR, Swadge_Parts:SOT-23-5, symbol Swadge_Parts:GS321-TR
- removed U9: GENERIC_LDO_1.8, Swadge_Parts:SOT-23, symbol Swadge_Parts:GENERIC_LDO_GOI
- added C25: 0.1μF, Swadge_Parts:C_0603_1608Metric, symbol Swadge_Parts:C
- added D11: D, Swadge_Parts:D_SMA, symbol Swadge_Parts:D
- added J1: LED, Swadge_Parts:PinHeader_1x03_P2.54mm_Vertical, symbol Swadge_Parts:Conn_01x03_Male
- added J2: DEBUG, Connector_PinHeader_2.54mm:PinHeader_2x10_P2.54mm_Vertical, symbol Connector_Generic:Conn_02x10_Odd_Even
- added L1: 33uH_500mA, Swadge_Parts:L_1210_3225Metric, symbol Swadge_Parts:L
- added MK2: N/A, Swadge_Parts:INGHAi GMI6050P-56DB, symbol Swadge_Parts:Microphone
- added Q1: PMOS, Package_TO_SOT_SMD:SOT-23, symbol Device:Q_PMOS_GSD
- added R2: 10Ω, Swadge_Parts:R_0603_1608Metric, symbol Swadge_Parts:R_US
- added R3: 2.2k, Swadge_Parts:R_0603_1608Metric, symbol Swadge_Parts:R_US
- C10: value 0.22μF -> .22μF
- C11: value 0.01μF -> .22μF; LCSC C14663 -> C21120
- C12, C13, C14, C15, C8: value 22μF -> .22μF; LCSC C86295 -> C21120
- C18: value 0.1μF -> .22μF; LCSC C282519 -> C21120
- C19: value 0.1μF -> 1μF; LCSC C282519 -> C1592
- C21: value 22μF -> 10μF; LCSC C86295 -> C96446
- C23: value 22μF -> 0.1μF; LCSC C86295 -> C282519
- C9: value 0.22μF -> 0.01μF; LCSC C21120 -> C14663
- D10, D5, D6, D7: value SK6812SIDE -> SK6812DSIDE; footprint Swadge_Parts:SK6812_SIDE_2 -> Swadge_Parts:SK6812D_SIDE; Digikey 1528-4691-ND -> (none); LCSC C2890037 -> C2890041
- MK1: footprint Swadge_Parts:INGHAi GMI6050P-56DB -> Swadge_Parts:GOERTEK_MIC_B4013AM423; Cost100 70 -> 13; Digikey 102-1721-ND -> N/A
- R5: value 47kΩ -> 100kΩ; LCSC C25819 -> C22936
- R6: value 10kΩ -> 43kΩ; LCSC C25197 -> C23172
- R8: value 10kΩ -> 0Ω; LCSC C25197 -> C15402
- R9: value 220kΩ -> 0Ω; LCSC C22939 -> C15402
Connections:
- net +3V3: now also R7.1, J2.16 (Pin_16), Q1.2 (S), R2.1; no longer U15.4 (VDD)
- net +5V: now also J2.18 (Pin_18)
- net 5VIN: now also J1.3 (Pin_3), J2.17 (Pin_17)
- net BATTPLUS: now also J2.15 (Pin_15)
- net BTN_1: now also C8.1; no longer C12.1
- net BTN_2: now also C10.1; no longer C13.1
- net BTN_3: now also C11.1; no longer C14.1
- net BTN_4: now also C13.1; no longer C15.2
- net BTN_5: now also C14.1; no longer C20.1
- net BTN_6: now also C15.1, U1.12 (GPIO8/TOUCH8/ADC1_CH7); no longer C21.1, U1.7 (GPIO7/TOUCH7/ADC1_CH6)
- net BTN_7: now also C12.1; no longer C22.1
- net BTN_8: now also C18.1; no longer C23.1
- net BZR: now also J2.2 (Pin_2)
- net GND: now also C10.2, C11.2, C15.2, C8.2, R6.2, R9.1, C25.2, D11.2 (A), J1.1 (Pin_1), J2.10 (Pin_10), J2.9 (Pin_9), MK2.1 (-); no longer C15.1, C21.2, C8.1, R6.1
- net LCD18: now also R8.1; no longer C18.1
- net LCD28: now also C23.1, R8.2, U10.2 (OUT), U15.4 (VDD), C25.1, J2.14 (Pin_14)
- net LED: now also J2.1 (Pin_1)
- net LED_OUT: now also J1.2 (Pin_2)
- net MIC: now also C21.2, C9.2, R5.2, R6.1, U1.7 (GPIO7/TOUCH7/ADC1_CH6); no longer C11.1, R9.1, U1.12 (GPIO8/TOUCH8/ADC1_CH7)
- net TFTATP: now also R7.2, Q1.1 (G)
- net TFT_CS: now also J2.6 (Pin_6)
- net TFT_FMARK: now also J2.11 (Pin_11)
- net TFT_LEDA: now also C22.1, J2.13 (Pin_13), L1.2
- net TFT_LEDK: now also R9.2
- net TFT_RESET: now also J2.12 (Pin_12)
- net TFT_RS: now also J2.5 (Pin_5)
- net TFT_SCL: now also J2.8 (Pin_8)
- net TFT_SDA: now also J2.7 (Pin_7)
- net GPIO17: now reaches U1.10 (GPIO17/U1TXD/ADC2_CH6/DAC_1)
- net GPIO17: now also J2.20 (Pin_20)
- net GPIO3: now reaches U1.15 (GPIO3/TOUCH3/ADC1_CH2)
- net GPIO3: now also J2.3 (Pin_3)
- net GPIO41: now reaches U1.34 (MTDI/GPIO41/CLK_OUT1)
- net GPIO41: now also J2.4 (Pin_4)
- net SNODE: now reaches C7.1, R21.2, SW9.2 (B), U3.1 (EN), U3.4 (VIN)
- net SNODE: now also J2.19 (Pin_19)
- net at R5.1: now also C20.1, R2.2, R3.1; no longer R6.2
- net TFTATN: no longer names the net of U1.24 (SPIIO4/GPIO33/FSPIHD)
- new net: D11.1 (K), L1.1, Q1.3 (D)
- new net: C21.1, MK1.2 (+), MK2.2 (+), R3.2
- no-connect marks 25 -> 22
Other:
- note added: "P-Mode Buck"
- note added: "TODO Use other footprint for LEDs"
- note removed: "TODO: Try 50dB+ Mic"
- note removed: "Two-Switch Buck-Boost"
- moved on the sheet: C16, C17, R26, U10

Commit message: update design
Parts:
- added J?: PGM, Connector_PinHeader_2.54mm:PinHeader_1x05_P2.54mm_Vertical, symbol Connector_Generic:Conn_01x05
- R8, R9: LCSC C15402 -> C21189
Connections:
- net 5VIN: now also J?.2 (Pin_2)
- net BTN_1: now also J?.1 (Pin_1)
- net GND: now also J?.5 (Pin_5)
- net LCD18: now also C25.1
- net LCD28: no longer C25.1
- net RX: now also J?.4 (Pin_4)
- net TX: now also J?.3 (Pin_3)
Changed lines of the file:
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@@
     )
   )
-  (global_label "LCD28" (shape input) (at 300.228 38.608 90) (fields_autoplaced)
-    (effects (font (size 1.27 1.27)) (justify left))
-    (property "Intersheet References" "${INTERSHEET_REFS}" (id 0) (at 300.3074 30.2078 90)
-      (effects (font (size 1.27 1.27)) (justify left) hide)
-    )
-  )
   (global_label "TOUCH_3" (shape input) (at 175.26 151.13 180) (fields_autoplaced)
     (effects (font (size 1.27 1.27)) (justify right))
@@
     )
   )
+  (global_label "5VIN" (shape input) (at 267.208 71.12 180) (fields_autoplaced)
+    (effects (font (size 1.27 1.27)) (justify right))
+    (property "Intersheet References" "${INTERSHEET_REFS}" (id 0) (at 260.5616 71.1994 0)
+      (effects (font (size 1.27 1.27)) (justify right) hide)
+    )
+  )
   (global_label "LCD28" (shape input) (at 309.372 149.86 0) (fields_autoplaced)
     (effects (font (size 1.27 1.27)) (justify left))
@@
     )
   )
+  (global_label "TX" (shape input) (at 267.208 73.66 180) (fields_autoplaced)
+    (effects (font (size 1.27 1.27)) (justify right))
+    (property "Intersheet References" "${INTERSHEET_REFS}" (id 0) (at 262.6178 73.7394 0)
+      (effects (font (size 1.27 1.27)) (justify right) hide)
+    )
+  )
   (global_label "TOUCH_1" (shape input) (at 44.45 59.69 180) (fields_autoplaced)
     (effects (font (size 1.27 1.27)) (justify right))
@@
     )
   )
+  (global_label "RX" (shape input) (at 267.208 76.2 180) (fields_autoplaced)
+    (effects (font (size 1.27 1.27)) (justify right))
+    (property "Intersheet References" "${INTERSHEET_REFS}" (id 0) (at 262.3154 76.2794 0)
+      (effects (font (size 1.27 1.27)) (justify right) hide)
+    )
+  )
   (global_label "TFT_RS" (shape input) (at 302.26 73.66 180) (fields_autoplaced)
     (effects (font (size 1.27 1.27)) (justify right))
@@
     )
   )
+  (global_label "LCD18" (shape input) (at 300.228 38.608 90) (fields_autoplaced)
+    (effects (font (size 1.27 1.27)) (justify left))
+    (property "Intersheet References" "${INTERSHEET_REFS}" (id 0) (at 300.3074 30.2078 90)
+      (effects (font (size 1.27 1.27)) (justify left) hide)
+    )
+  )
   (global_label "TFT_CS" (shape input) (at 302.26 71.12 180) (fields_autoplaced)
     (effects (font (size 1.27 1.27)) (justify right))
@@
     )
   )
+  (global_label "BTN_1" (shape input) (at 267.208 68.58 180) (fields_autoplaced)
+    (effects (font (size 1.27 1.27)) (justify right))
+    (property "Intersheet References" "${INTERSHEET_REFS}" (id 0) (at 259.0497 68.5006 0)
+      (effects (font (size 1.27 1.27)) (justify right) hide)
+    )
+  )
   (global_label "LCD18" (shape input) (at 321.31 71.12 0) (fields_autoplaced)
     (effects (font (size 1.27 1.27)) (justify left))
@@
       (effects (font (size 1.27 1.27)) hide)
     )
-    (property "LCSC" "C15402" (id 7) (at 325.12 106.426 0)
+    (property "LCSC" "C21189" (id 7) (at 325.12 106.426 0)
       (effects (font (size 1.27 1.27)) hide)
     )
@@
     (pin "1")
   )
+  (symbol (lib_id "Connector_Generic:Conn_01x05") (at 272.288 73.66 0) (unit 1)
+    (in_bom yes) (on_board yes) (fields_autoplaced)
+    (property "Reference" "J?" (id 0) (at 274.32 72.8253 0)
+      (effects (font (size 1.27 1.27)) (justify left))
+    )
+    (property "Value" "PGM" (id 1) (at 274.32 75.3622 0)
+      (effects (font (size 1.27 1.27)) (justify left))
+    )
+    (property "Footprint" "Connector_PinHeader_2.54mm:PinHeader_1x05_P2.54mm_Vertical" (id 2) (at 272.288 73.66 0)
+      (effects (font (size 1.27 1.27)) hide)
+    )
+    (property "Datasheet" "~" (id 3) (at 272.288 73.66 0)
+      (effects (font (size 1.27 1.27)) hide)
+    )
+    (property "LCSC" "NP" (id 4) (at 272.288 73.66 0)
+      (effects (font (size 1.27 1.27)) hide)
+    )
+    (pin "1")
+    (pin "2")
+    (pin "3")
+    (pin "4")
+    (pin "5")
+  )
   (symbol (lib_id "Swadge_Parts:Microphone") (at 238.125 42.545 0) (unit 1)
     (in_bom yes) (on_board yes)
@@
     (pin "1")
   )
+  (symbol (lib_id "Swadge_Parts:GND") (at 267.208 78.74 270) (unit 1)
+    (in_bom yes) (on_board yes)
+    (property "Reference" "#PWR?" (id 0) (at 260.858 78.74 0)
+      (effects (font (size 1.27 1.27)) hide)
+    )
+    (property "Value" "GND" (id 1) (at 262.382 78.994 90))
+    (property "Footprint" "" (id 2) (at 267.208 78.74 0)
+      (effects (font (size 1.27 1.27)) hide)
+    )
+    (property "Datasheet" "" (id 3) (at 267.208 78.74 0)
+      (effects (font (size 1.27 1.27)) hide)
+    )
+    (pin "1")
+  )
   (symbol (lib_name "SK6812SIDE_2") (lib_id "Swadge_Parts:SK6812SIDE") (at 41.91 138.43 0) (unit 1)
     (in_bom yes) (on_board yes)
@@
       (effects (font (size 1.27 1.27)) hide)
     )
-    (property "LCSC" "C15402" (id 7) (at 323.85 139.7 0)
+    (property "LCSC" "C21189" (id 7) (at 323.85 139.7 0)
       (effects (font (size 1.27 1.27)) hide)
     )
@@
       (reference "#PWR0116") (unit 1) (value "GND") (footprint "")
     )
+    (path "/b0c4b47b-f7ae-4d66-b619-e92865675556"
+      (reference "#PWR?") (unit 1) (value "GND") (footprint "")
+    )
     (path "/6efbac4e-4c48-4d85-b138-3166666d2e76"
       (reference "BT1") (unit 1) (value "Battery") (footprint "Swadge_Parts:2460")
@@
       (reference "J2") (unit 1) (value "DEBUG") (footprint "Connector_PinHeader_2.54mm:PinHeader_2x10_P2.54mm_Vertical")
     )
+    (path "/a55c1b99-3293-490d-831c-cf15a08bdfa8"
+      (reference "J?") (unit 1) (value "PGM") (footprint "Connector_PinHeader_2.54mm:PinHeader_1x05_P2.54mm_Vertical")
+    )
     (path "/3e011cdb-c151-46b2-9f97-ba78518661fd"
